File: kicad/ch32v3x/lnBMP_ch32/lnBMP_ch32.kicad_sch (KiCad schematic)
At the start: 19 parts

Commit message: update schematic for ch32
Parts:
- added R? (x2): 1k, symbol Device:R_Small
Connections:
- net GND: now also R?.1
- net at U?.17 (PA3): now also R?.2, R?.2
- net OUT_NRESET renamed INOUT_NRESET
- net INOUT_NRESET: now also R?.1
Changed lines of the file:
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@@
   (junction (at 265.43 24.13) (diameter 0) (color 0 0 0 0)
   )
+  (junction (at 91.44 74.93) (diameter 0) (color 0 0 0 0)
+  )
   (junction (at 252.73 31.75) (diameter 0) (color 0 0 0 0)
   )
@@
   )
   (wire (pts (xy 69.85 153.67) (xy 69.85 156.21))
+    (stroke (width 0) (type default) (color 0 0 0 0))
+  )
+  (wire (pts (xy 86.36 74.93) (xy 91.44 74.93))
     (stroke (width 0) (type default) (color 0 0 0 0))
   )
@@
     )
   )
-  (global_label "OUT_NRESET" (shape output) (at 88.9 125.73 0) (fields_autoplaced)
-    (effects (font (size 1.27 1.27)) (justify left))
-    (property "Intersheet References" "${INTERSHEET_REFS}" (id 0) (at 102.985 125.6506 0)
+  (global_label "INOUT_NRESET" (shape bidirectional) (at 88.9 125.73 0) (fields_autoplaced)
+    (effects (font (size 1.27 1.27)) (justify left))
+    (property "Intersheet References" "${INTERSHEET_REFS}" (id 0) (at 104.9202 125.6506 0)
       (effects (font (size 1.27 1.27)) (justify left) hide)
     )
@@
     )
   )
-  (global_label "OUT_NRESET" (shape input) (at 133.35 80.01 180) (fields_autoplaced)
+  (global_label "INOUT_NRESET" (shape bidirectional) (at 133.35 80.01 180) (fields_autoplaced)
     (effects (font (size 1.27 1.27)) (justify right))
-    (property "Intersheet References" "${INTERSHEET_REFS}" (id 0) (at 119.265 79.9306 0)
+    (property "Intersheet References" "${INTERSHEET_REFS}" (id 0) (at 117.3298 79.9306 0)
       (effects (font (size 1.27 1.27)) (justify right) hide)
     )
@@
     (property "Intersheet References" "${INTERSHEET_REFS}" (id 0) (at 137.0806 159.3488 90)
       (effects (font (size 1.27 1.27)) (justify right) hide)
+    )
+  )
+  (global_label "INOUT_NRESET" (shape bidirectional) (at 96.52 74.93 0) (fields_autoplaced)
+    (effects (font (size 1.27 1.27)) (justify left))
+    (property "Intersheet References" "${INTERSHEET_REFS}" (id 0) (at 112.5402 74.8506 0)
+      (effects (font (size 1.27 1.27)) (justify left) hide)
     )
   )
@@
     (pin "2")
   )
+  (symbol (lib_id "Device:R_Small") (at 91.44 77.47 180) (unit 1)
+    (in_bom yes) (on_board yes)
+    (property "Reference" "R?" (id 0) (at 92.71 77.47 0)
+      (effects (font (size 1.27 1.27)) (justify right))
+    )
+    (property "Value" "1k" (id 1) (at 92.71 80.01 0)
+      (effects (font (size 1.27 1.27)) (justify right))
+    )
+    (property "Footprint" "" (id 2) (at 91.44 77.47 0)
+      (effects (font (size 1.27 1.27)) hide)
+    )
+    (property "Datasheet" "~" (id 3) (at 91.44 77.47 0)
+      (effects (font (size 1.27 1.27)) hide)
+    )
+    (pin "1")
+    (pin "2")
+  )
+  (symbol (lib_id "power:GND") (at 91.44 80.01 0) (unit 1)
+    (in_bom yes) (on_board yes) (fields_autoplaced)
+    (property "Reference" "#PWR?" (id 0) (at 91.44 86.36 0)
+      (effects (font (size 1.27 1.27)) hide)
+    )
+    (property "Value" "GND" (id 1) (at 91.44 85.09 0))
+    (property "Footprint" "" (id 2) (at 91.44 80.01 0)
+      (effects (font (size 1.27 1.27)) hide)
+    )
+    (property "Datasheet" "" (id 3) (at 91.44 80.01 0)
+      (effects (font (size 1.27 1.27)) hide)
+    )
+    (pin "1")
+  )
   (symbol (lib_id "Connector:USB_OTG") (at 214.63 29.21 0) (unit 1)
     (in_bom yes) (on_board yes) (fields_autoplaced)
@@
     (pin "1")
   )
+  (symbol (lib_id "Device:R_Small") (at 93.98 74.93 270) (unit 1)
+    (in_bom yes) (on_board yes)
+    (property "Reference" "R?" (id 0) (at 93.98 69.85 90))
+    (property "Value" "1k" (id 1) (at 93.98 72.39 90))
+    (property "Footprint" "" (id 2) (at 93.98 74.93 0)
+      (effects (font (size 1.27 1.27)) hide)
+    )
+    (property "Datasheet" "~" (id 3) (at 93.98 74.93 0)
+      (effects (font (size 1.27 1.27)) hide)
+    )
+    (pin "1")
+    (pin "2")
+  )
   (symbol (lib_id "power:+3.3V") (at 38.1 35.56 0) (unit 1)
     (in_bom yes) (on_board yes) (fields_autoplaced)
@@
       (reference "#PWR?") (unit 1) (value "GND") (footprint "")
     )
+    (path "/babcada7-9572-4b74-bda5-efcb24966f5a"
+      (reference "#PWR?") (unit 1) (value "GND") (footprint "")
+    )
     (path "/c8f06c19-b88f-45dc-8569-1e336ed34746"
       (reference "#PWR?") (unit 1) (value "GND") (footprint "")
@@
       (reference "R?") (unit 1) (value "10k") (footprint "")
     )
+    (path "/ba1855e9-d148-40ee-ba64-5574c8462282"
+      (reference "R?") (unit 1) (value "1k") (footprint "")
+    )
     (path "/c9e215f6-7d50-4fb7-961d-1e6c48f6750e"
       (reference "R?") (unit 1) (value "330") (footprint "")
     )
+    (path "/ec1e9184-2829-4a0c-b23d-b678c7ab127f"
+      (reference "R?") (unit 1) (value "1k") (footprint "")
+    )
     (path "/157e8597-0dfe-461a-be75-d90ba0ece56b"

Commit message: update kicar
Parts:
- removed D?: LED, symbol Device:LED
- added C6, C7, C8, C9: 100n, Capacitor_SMD:C_0402_1005Metric, symbol Device:C_Small
- C1, C2, C3, C5: renamed from C?; footprint (none) -> Capacitor_SMD:C_0402_1005Metric
- C4: renamed from C?; footprint (none) -> Capacitor_THT:CP_Radial_D4.0mm_P2.00mm
- D1: renamed from D?; footprint (none) -> Diode_SMD:D_0805_2012Metric
- J1, J2, J3: renamed from J?; footprint (none) -> Connector_JST:JST_XH_B4B-XH-A_1x04_P2.50mm_Vertical
- J4: renamed from J?; footprint (none) -> Connector_USB:USB_Mini-B_Lumberg_2486_01_Horizontal
- R1, R2, R3, R4, R5: renamed from R?; footprint (none) -> Resistor_SMD:R_0402_1005Metric
- SW1, SW2: renamed from SW?; footprint (none) -> Button_Switch_SMD:SW_SPST_B3U-3000P-B
- U2: renamed from U?; footprint (none) -> Package_TO_SOT_SMD:SOT-223
- Y1: renamed from Y?; footprint (none) -> Crystal:Crystal_HC49-U_Vertical
- gave numbers to parts that had none: 1
Connections:
- net +3.3V: now also C6.1, C7.1, C8.1, C9.1
- net GND: now also C6.2, C7.2, C8.2, C9.2

Commit message: update kicad
Parts:
- J4: footprint Connector_USB:USB_Mini-B_Lumberg_2486_01_Horizontal -> Connector_USB:USB_Micro-B_Wuerth_629105150521
Changed lines of the file:
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@@
       (effects (font (size 1.27 1.27)))
     )
-    (property "Footprint" "Connector_USB:USB_Mini-B_Lumberg_2486_01_Horizontal" (at 218.44 30.48 0)
+    (property "Footprint" "Connector_USB:USB_Micro-B_Wuerth_629105150521" (at 218.44 30.48 0)
       (effects (font (size 1.27 1.27)) hide)
     )

Commit message: update CH32 PCB to rev B
Parts:
- BOT1: renamed from SW1; footprint Button_Switch_SMD:SW_SPST_B3U-3000P-B -> Button_Switch_SMD:SW_SPST_CK_RS282G05A3
- C1, C2, C3, C5, C6, C7, C8, C9: footprint Capacitor_SMD:C_0402_1005Metric -> Resistor_SMD:R_0603_1608Metric
- R1, R2, R3, R4, R5: footprint Resistor_SMD:R_0402_1005Metric -> Resistor_SMD:R_0603_1608Metric
- RST1: renamed from SW2; footprint Button_Switch_SMD:SW_SPST_B3U-3000P-B -> Button_Switch_SMD:SW_SPST_CK_RS282G05A3
Connections:
- net UART TX is gone; now on net UART_TX: J3.4 (Pin_4)
Changed lines of the file:
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@@
     )
   )
-  (global_label "UART TX" (shape input) (at 139.7 149.86 270) (fields_autoplaced)
+  (global_label "UART_TX" (shape input) (at 139.7 149.86 270) (fields_autoplaced)
     (effects (font (size 1.27 1.27)) (justify right))
-    (property "Intersheetrefs" "${INTERSHEET_REFS}" (at 139.6206 160.0745 90)
+    (property "Intersheetrefs" "${INTERSHEET_REFS}" (at 139.7 160.5672 90)
       (effects (font (size 1.27 1.27)) (justify right) hide)
     )
@@
       (effects (font (size 1.27 1.27)) (justify left))
     )
-    (property "Footprint" "Capacitor_SMD:C_0402_1005Metric" (at 106.68 39.37 0)
+    (property "Footprint" "Resistor_SMD:R_0603_1608Metric" (at 106.68 39.37 0)
       (effects (font (size 1.27 1.27)) hide)
     )
@@
       (effects (font (size 1.27 1.27)))
     )
-    (property "Footprint" "Capacitor_SMD:C_0402_1005Metric" (at 39.37 100.33 0)
+    (property "Footprint" "Resistor_SMD:R_0603_1608Metric" (at 39.37 100.33 0)
       (effects (font (size 1.27 1.27)) hide)
     )
@@
   (symbol (lib_id "Switch:SW_DIP_x01") (at 38.1 52.07 270) (unit 1)
     (in_bom yes) (on_board yes) (dnp no) (fields_autoplaced)
-    (property "Reference" "SW2" (at 45.72 52.07 0)
-      (effects (font (size 1.27 1.27)))
-    )
-    (property "Value" "SW_DIP_x01" (at 43.18 52.07 0)
-      (effects (font (size 1.27 1.27)))
-    )
-    (property "Footprint" "Button_Switch_SMD:SW_SPST_B3U-3000P-B" (at 38.1 52.07 0)
+    (property "Reference" "RST1" (at 41.91 50.8 90)
+      (effects (font (size 1.27 1.27)) (justify left))
+    )
+    (property "Value" "SW_DIP_x01" (at 41.91 53.34 90)
+      (effects (font (size 1.27 1.27)) (justify left))
+    )
+    (property "Footprint" "Button_Switch_SMD:SW_SPST_CK_RS282G05A3" (at 38.1 52.07 0)
       (effects (font (size 1.27 1.27)) hide)
     )
@@
       (project "lnBMP_ch32"
         (path "/fbe443d6-6d74-4abc-9dee-16e0160553bc"
-          (reference "SW2") (unit 1)
+          (reference "RST1") (unit 1)
         )
       )
@@
       (effects (font (size 1.27 1.27)) (justify left))
     )
-    (property "Footprint" "Resistor_SMD:R_0402_1005Metric" (at 20.32 54.61 0)
+    (property "Footprint" "Resistor_SMD:R_0603_1608Metric" (at 20.32 54.61 0)
       (effects (font (size 1.27 1.27)) hide)
     )
@@
       (effects (font (size 1.27 1.27)) (justify left))
     )
-    (property "Footprint" "Capacitor_SMD:C_0402_1005Metric" (at 113.03 39.37 0)
+    (property "Footprint" "Resistor_SMD:R_0603_1608Metric" (at 113.03 39.37 0)
       (effects (font (size 1.27 1.27)) hide)
     )
@@
       (effects (font (size 1.27 1.27)) (justify left))
     )
-    (property "Footprint" "Capacitor_SMD:C_0402_1005Metric" (at 265.43 26.67 0)
+    (property "Footprint" "Resistor_SMD:R_0603_1608Metric" (at 265.43 26.67 0)
       (effects (font (size 1.27 1.27)) hide)
     )
@@
       (effects (font (size 1.27 1.27)) (justify left))
     )
-    (property "Footprint" "Capacitor_SMD:C_0402_1005Metric" (at 99.06 39.37 0)
+    (property "Footprint" "Resistor_SMD:R_0603_1608Metric" (at 99.06 39.37 0)
       (effects (font (size 1.27 1.27)) hide)
     )
@@
       (effects (font (size 1.27 1.27)) (justify left))
     )
-    (property "Footprint" "Resistor_SMD:R_0402_1005Metric" (at 38.1 38.1 0)
+    (property "Footprint" "Resistor_SMD:R_0603_1608Metric" (at 38.1 38.1 0)
       (effects (font (size 1.27 1.27)) hide)
     )
@@
       (effects (font (size 1.27 1.27)) (justify left))
     )
-    (property "Footprint" "Capacitor_SMD:C_0402_1005Metric" (at 92.71 39.37 0)
+    (property "Footprint" "Resistor_SMD:R_0603_1608Metric" (at 92.71 39.37 0)
       (effects (font (size 1.27 1.27)) hide)
     )
@@
       (effects (font (size 1.27 1.27)) (justify left))
     )
-    (property "Footprint" "Capacitor_SMD:C_0402_1005Metric" (at 30.48 52.07 0)
+    (property "Footprint" "Resistor_SMD:R_0603_1608Metric" (at 30.48 52.07 0)
       (effects (font (size 1.27 1.27)) hide)
     )
@@
       (effects (font (size 1.27 1.27)) (justify right))
     )
-    (property "Footprint" "Resistor_SMD:R_0402_1005Metric" (at 91.44 77.47 0)
+    (property "Footprint" "Resistor_SMD:R_0603_1608Metric" (at 91.44 77.47 0)
       (effects (font (size 1.27 1.27)) hide)
     )
@@
       (effects (font (size 1.27 1.27)))
     )
-    (property "Footprint" "Resistor_SMD:R_0402_1005Metric" (at 43.18 143.51 0)
+    (property "Footprint" "Resistor_SMD:R_0603_1608Metric" (at 43.18 143.51 0)
       (effects (font (size 1.27 1.27)) hide)
     )
@@
       (effects (font (size 1.27 1.27)))
     )
-    (property "Footprint" "Capacitor_SMD:C_0402_1005Metric" (at 39.37 92.71 0)
+    (property "Footprint" "Resistor_SMD:R_0603_1608Metric" (at 39.37 92.71 0)
       (effects (font (size 1.27 1.27)) hide)
     )
@@
   (symbol (lib_id "Switch:SW_DIP_x01") (at 20.32 64.77 270) (unit 1)
     (in_bom yes) (on_board yes) (dnp no) (fields_autoplaced)
-    (property "Reference" "SW1" (at 27.94 64.77 0)
-      (effects (font (size 1.27 1.27)))
-    )
-    (property "Value" "SW_DIP_x01" (at 25.4 64.77 0)
-      (effects (font (size 1.27 1.27)))
-    )
-    (property "Footprint" "Button_Switch_SMD:SW_SPST_B3U-3000P-B" (at 20.32 64.77 0)
+    (property "Reference" "BOT1" (at 24.13 63.5 90)
+      (effects (font (size 1.27 1.27)) (justify left))
+    )
+    (property "Value" "SW_DIP_x01" (at 24.13 66.04 90)
+      (effects (font (size 1.27 1.27)) (justify left))
+    )
+    (property "Footprint" "Button_Switch_SMD:SW_SPST_CK_RS282G05A3" (at 20.32 64.77 0)
       (effects (font (size 1.27 1.27)) hide)
     )
@@
       (project "lnBMP_ch32"
         (path "/fbe443d6-6d74-4abc-9dee-16e0160553bc"
-          (reference "SW1") (unit 1)
+          (reference "BOT1") (unit 1)
         )
       )
@@
       (effects (font (size 1.27 1.27)))
     )
-    (property "Footprint" "Resistor_SMD:R_0402_1005Metric" (at 93.98 74.93 0)
-      (effects (font (size 1.27 1.27)) hide)
-    )
+    (property "Footprint" "Resistor_SMD:R_0603_1608Metric" (at 93.98 74.93 0)
+      (effects (font (size 1.27 1.27)) hide)
+    )

Commit message: update ch32 pcba
Connections:
- net IN_FORCE_DFU: now reaches U1.35 (PB14)
Changed lines of the file:
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@@
+    (stroke (width 0) (type default))
+  )
+  (wire (pts (xy 86.36 146.05) (xy 88.9 146.05))
     (stroke (width 0) (type default))
   )
@@
       (effects (font (size 1.27 1.27)) (justify left) hide)
     )
+  )
+  (global_label "IN_FORCE_DFU" (shape output) (at 88.9 146.05 0) (fields_autoplaced)
+    (effects (font (size 1.27 1.27)) (justify left))
+    (property "Intersheetrefs" "${INTERSHEET_REFS}" (at 105.4735 146.05 0)
+      (effects (font (size 1.27 1.27)) (justify left) hide)
+    )

Commit message: kicad : Update ch32 and stm32 pcbs
Parts:
- R4, R5: value 1k -> 10k
Changed lines of the file:
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@@
     (effects (font (size 1.27 1.27)) (justify right))
     (property "Intersheetrefs" "${INTERSHEET_REFS}" (at 119.9818 66.04 0)
-      (effects (font (size 1.27 1.27)) (justify right))
+      (effects (font (size 1.27 1.27)) (justify right) hide)
     )
   )
@@
       (effects (font (size 1.27 1.27)) (justify right))
     )
-    (property "Value" "1k" (at 92.71 80.01 0)
+    (property "Value" "10k" (at 92.71 80.01 0)
       (effects (font (size 1.27 1.27)) (justify right))
     )
@@
       (effects (font (size 1.27 1.27)))
     )
-    (property "Value" "1k" (at 93.98 72.39 90)
-      (effects (font (size 1.27 1.27)))
-    )
+    (property "Value" "10k" (at 93.98 72.39 90)
+      (effects (font (size 1.27 1.27)))
+    )
