File: kicad/ch32v3x/lnBMP_ch32d/lnBMP_ch32revD/lnBMP_ch32revC.kicad_pcb (KiCad board)
At the start: 2 copper layers, 52.6 x 33 mm, 29 parts, among them J1 BMP Debug1, J2 BMP Debug2, J3 Debug port, J4 USB_OTG, U1 CH32V303RCT6, U2 LM1117-3.3, Y1 Crystal, x2 PinSocket_1x03_P1.00mm_Vertic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

Commit message: new rev of ch32 pcb
Parts:
- moved x2 3.62 mm to (140.9, 86.1)
- moved R5 3.60 mm to (120.6, 93.8)
- moved J2 2.55 mm to (109.1, 88.4)
- moved J1 2.42 mm to (109.1, 70.5)
- moved R3 1.24 mm to (138.7, 93.8)
- moved D1 1.08 mm to (142.9, 93.6)
- moved C6 0.76 mm to (134.2, 95.8)
- moved J3 0.39 mm to (142.1, 71.2)
- moved 3/3/GND/GND 0.20 mm to (137.3, 96.7)
- moved x 0.20 mm to (121.6, 91.4)
Routing:
- net INOUT_NRESET: track 54.6 -> 47.4 mm
- net GND: track 223.5 -> 216.5 mm
- net Net-(U1-PA3): track 3.12 -> 6.83 mm
- net unconnected-(U1-PC11-Pad52): track 2.75 -> 0.00 mm, vias 1 -> 0
- net Net-(J4-VBUS): track 25.8 -> 23.4 mm
- net OUT_UART_RX: track 29.9 -> 27.9 mm
- net UART_TX: track 12.6 -> 10.8 mm
- net OUT_SWDIO: track 27.4 -> 25.8 mm
- net OUT_SWDCLK: track 25.4 -> 23.8 mm
- net +3.3V: track 136.4 -> 137.9 mm
- net OUT_UART_TX: track 33.8 -> 35.3 mm
- net Net-(U1-PC13): track 19.0 -> 17.7 mm
- net SWDIO: track 12.3 -> 11.4 mm
- net D-: track 18.0 -> 18.8 mm
- net D+: track 17.9 -> 18.7 mm
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Other:
- board size 52.6 x 33 mm -> 51 x 33.3 mm
- board text added: "CK"
- board text added: "GD"
- board text added: "IO"
- board text added: "REVD"
- board text removed: "REVB"
- board text removed: "SWDCLK"
- board text removed: "SWDIO"

Commit message: pcb/ch32: reduce R5
Parts:
- R5: value 10k -> 1k

Commit message: kicad: update ch32 pcb to revD
Parts:
- added kibuzzard-6534F5CB: G***, kibuzzard-6534F5CB, F.Cu at (113.6, 75.1)
- added kibuzzard-6534F635: G***, kibuzzard-6534F635, F.Cu at (113.4, 73.0)
- added kibuzzard-6534F652: G***, kibuzzard-6534F652, F.Cu at (114.5, 78.2)
- added kibuzzard-6534F67C: G***, kibuzzard-6534F67C, F.Cu at (112.9, 86.3)
- added kibuzzard-6534F68E: G***, kibuzzard-6534F68E, F.Cu at (115.3, 93.6)
- added kibuzzard-6534F6A3: G***, kibuzzard-6534F6A3, F.Cu at (115.4, 92.0)
- added kibuzzard-6534F6BC: G***, kibuzzard-6534F6BC, F.Cu at (112.9, 95.7)
- added kibuzzard-6534F8DC: G***, kibuzzard-6534F8DC, F.Cu at (135.0, 72.9)
- added kibuzzard-6534F8F1: G***, kibuzzard-6534F8F1, F.Cu at (135.0, 74.1)
- added kibuzzard-6534F8FD: G***, kibuzzard-6534F8FD, F.Cu at (135.0, 76.0)
- added kibuzzard-6534F90C: G***, kibuzzard-6534F90C, F.Cu at (135.3, 77.4)
- added kibuzzard-6534F947: G***, kibuzzard-6534F947, F.Cu at (143.0, 87.1)
Other:
- board text removed: "locked"

Commit message: kicad/ch32: Fix swapped labels, orienttion
Parts:
- added DFU1: SWDFU, Button_Switch_SMD:SW_SPST_CK_RS282G05A3, F.Cu at (4.92, 2.08)
- moved J3 7.56 mm to (142.1, 78.8), turned to 90 degrees
- moved kibuzzard-6534F8F1 2.06 mm to (135.8, 76.0)
- moved kibuzzard-6534F8FD 2.02 mm to (134.3, 74.1)
Connections:
- J3 pad 1: GND -> UART_TX
- J3 pad 2: SWDCLK -> SWDIO
- J3 pad 3: SWDIO -> SWDCLK
- J3 pad 4: UART_TX -> GND
