File: kicad/ch32v3x/lnBMP_ch32f/lnBMP_ch32revF/lnBMP_ch32revF.kicad_pcb (KiCad board)
At the start: 2 copper layers, 51 x 33.3 mm, 52 parts, among them J1 BMP Debug1, J2 BMP Debug2, J3 Debug port, J4 USB_C_Receptacle, U1 CH32V303RCT6, U2 LM1117-3.3, Y1 Crystal, x2 PinSocket_1x03_P1.00mm_Vertic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

Commit message: kicad : rev F fix rev name onboard
Parts:
- removed kibuzzard-65C2815C: G***, kibuzzard-65C2815C
- removed kibuzzard-65C283CB: G***, kibuzzard-65C283CB
- added kibuzzard-65D8420C: G***, kibuzzard-65D8420C, F.Cu at (130.1, 74.0)
- added kibuzzard-65D842E2: G***, kibuzzard-65D842E2, F.Cu at (118.5, 99.2)
