File: kicad/ch32v3x/lnBMP_ch32f_5pins/lnBMP_ch32_revF_5pins.kicad_sch (KiCad schematic)
At the start: 26 parts, among them J1 Conn_ARM_JTAG_SWD_10, J3 Debug port, J4 USB_C_Receptacle, J5 Debug port, U1 CH32V303RCT6, U2 LM1117-3.3, Y1 Crystal

Commit message: ch32: update a bit the pcb
Parts:
- removed BOT1: SW_DIP_x01, Button_Switch_SMD:SW_SPST_CK_RS282G05A3, symbol Switch:SW_DIP_x01
- R1: value 10k -> 1k
Connections:
- net +3.3V: no longer R1.1
- net GND: now also R1.2; no longer DFU1.2
- net IN_FORCE_DFU: now also DFU1.1, U1.59 (PB7); no longer U1.35 (PB14)
- net at R5.2: now also U1.20 (PA4); no longer U1.17 (PA3)
- net INOUT_SWO: now reaches J1.6 (SWO/TDO)
- net INOUT_SWO: now also U1.17 (PA3)
- new net: DFU1.2, R1.1
Other:
- moved on the sheet: DFU1, R1, R5
