File: kicad/ch32v3x/lnBMP_ch32f_5pins/lnBMP_ch32_revF_5pins.kicad_pcb (KiCad board)
At the start: 2 copper layers, 51 x 33.3 mm, 49 parts, among them J1 Conn_ARM_JTAG_SWD_10, J3 Debug port, J4 USB_C_Receptacle, J5 Debug port, U1 CH32V303RCT6, U2 LM1117-3.3, Y1 Crystal, x2 PinSocket_1x03_P1.00mm_Vertic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

Commit message: ch32: update a bit the pcb
Parts:
- removed BOT1: SW_DIP_x01, Button_Switch_SMD:SW_SPST_CK_RS282G05A3
- removed Rxx: 10k, Resistor_SMD:R_0603_1608Metric
- removed kibuzzard-6534F947: G***, kibuzzard-6534F947
- removed kibuzzard-65C1C9E5: G***, kibuzzard-65C1C9E5
- added DFU1: SWDFU, Button_Switch_SMD:SW_SPST_CK_RS282G05A3, F.Cu at (130.1, 69.7)
- added kibuzzard-664C331A: G***, kibuzzard-664C331A, F.Cu at (130.5, 72.4)
- R1: value 10k -> 1k
- moved R1 9.32 mm to (126.7, 73.2), turned to 180 degrees
- moved R2 3.20 mm to (120.7, 74.0)
- moved C1 1.80 mm to (123.3, 73.2), turned to 0 degrees
- moved R5 1.20 mm to (120.5, 95.1)
- moved x 1.02 mm to (121.6, 92.6)
- moved kibuzzard-65D8420C 1.00 mm to (131.1, 74.1)
- turned RST1 to 0 degrees
Connections:
- J1 pad 6: unconnected-(J1-SWO/TDO-Pad6) -> INOUT_SWO
- R1 pad 1: +3.3V -> Net-(DFU1-Pad2)
- R1 pad 2: Net-(BOT1-Pad1) -> GND
- R5 pad 2: Net-(U1-PA3) -> Net-(U1-PA4)
- U1 pad 17: Net-(U1-PA3) -> INOUT_SWO
- U1 pad 20: unconnected-(U1-PA4-Pad20) -> Net-(U1-PA4)
- U1 pad 35: IN_FORCE_DFU -> unconnected-(U1-PB14-Pad35)
- U1 pad 59: unconnected-(U1-PB7-Pad59) -> IN_FORCE_DFU
- U1 pad 60: Net-(U1-BOOT0) -> unconnected-(U1-BOOT0-Pad60)
- x2 pad 2: IN_FORCE_DFU -> unconnected-(U1-PB14-Pad35)
Routing:
- net INOUT_SWO: track 0.00 -> 23.9 mm, vias 0 -> 2
- net Net-(U1-BOOT0): track 12.3 -> 0.00 mm
- net IN_FORCE_DFU: track 5.54 -> 15.2 mm
- net Net-(U1-PA4): track 0.00 -> 8.95 mm
- net Net-(U1-PA3): track 7.15 -> 0.00 mm
- net unconnected-(U1-PB14-Pad35): track 0.00 -> 5.54 mm
- net unconnected-(U1-PA4-Pad20): track 4.50 -> 0.00 mm
- net Net-(DFU1-Pad2): track 0.00 -> 3.75 mm
- net +3.3V: track 136.3 -> 133.2 mm
- net Net-(BOT1-Pad1): track 1.12 -> 0.00 mm
- net unconnected-(U1-PA0-Pad14): track 4.36 -> 5.44 mm
- net NRESET: track 68.9 -> 69.8 mm
- net unconnected-(U1-PA1-Pad15): track 6.58 -> 7.55 mm
- net unconnected-(U1-PA2-Pad16): track 2.30 -> 2.97 mm
- net GND: track 208.9 -> 209.5 mm, vias 5 -> 7
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
Commit message: small ch32 pcb update
Parts:
- added kibuzzard-66C04316: G***, kibuzzard-66C04316, F.Cu at (111.5, 89.6)
- added kibuzzard-66C04342: G***, kibuzzard-66C04342, F.Cu at (107.4, 89.8)
- added kibuzzard-66C0434B: G***, kibuzzard-66C0434B, F.Cu at (105.7, 89.8)
- added kibuzzard-66C04372: G***, kibuzzard-66C04372, F.Cu at (111.0, 97.5)
- added kibuzzard-66C0437E: G***, kibuzzard-66C0437E, F.Cu at (108.5, 97.5)
- added kibuzzard-66C043C9: G***, kibuzzard-66C043C9, F.Cu at (108.5, 98.6)
Routing:
- net OUT_UART_RX: track 49.9 -> 46.2 mm
- net GND: track 209.5 -> 208.6 mm
- added copper zone on B.Cu, net GND
- added copper zone on F.Cu, net GND
