File: kicad/stm32f1/lnBMP_stm32_5pin_voltage_shifter2/mcu.kicad_sch (KiCad schematic)
At the start: 16 parts, among them J4 DFU, J5 BOOT, U1 GD32F303, Y2 8Mhz

Commit message: beginning GD32 version
Connections:
- net DP: now reaches R6.2, R7.2, U1.33 (PA12)
- net DN: now reaches R5.2, U1.32 (PA11)
Changed lines of the file:
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@@
+	)
+	(junction
+		(at 168.91 92.71)
+		(diameter 0)
+		(color 0 0 0 0)
 	)
 	(junction
@@
 	)
 	(junction
+		(at 189.23 97.79)
+		(diameter 0)
+		(color 0 0 0 0)
+	)
+	(junction
 		(at 87.63 46.99)
 		(diameter 0)
@@
 	(wire
 		(pts
+			(xy 180.34 90.17) (xy 180.34 85.09)
+		)
+		(stroke
+			(width 0)
+			(type default)
+		)
+	)
+	(wire
+		(pts
 			(xy 119.38 77.47) (xy 121.92 77.47)
 		)
@@
 	(wire
 		(pts
+			(xy 189.23 105.41) (xy 191.77 105.41)
+		)
+		(stroke
+			(width 0)
+			(type default)
+		)
+	)
+	(wire
+		(pts
 			(xy 107.95 40.64) (xy 107.95 41.91)
 		)
@@
 	(wire
 		(pts
+			(xy 168.91 92.71) (xy 168.91 90.17)
+		)
+		(stroke
+			(width 0)
+			(type default)
+		)
+	)
+	(wire
+		(pts
+			(xy 189.23 97.79) (xy 189.23 105.41)
+		)
+		(stroke
+			(width 0)
+			(type default)
+		)
+	)
+	(wire
+		(pts
 			(xy 96.52 88.9) (xy 104.14 88.9)
 		)
@@
 	(wire
 		(pts
+			(xy 168.91 90.17) (xy 180.34 90.17)
+		)
+		(stroke
+			(width 0)
+			(type default)
+		)
+	)
+	(wire
+		(pts
 			(xy 154.94 95.25) (xy 167.64 95.25)
 		)
@@
 	(wire
 		(pts
+			(xy 189.23 97.79) (xy 167.64 97.79)
+		)
+		(stroke
+			(width 0)
+			(type default)
+		)
+	)
+	(wire
+		(pts
 			(xy 120.65 64.77) (xy 121.92 64.77)
 		)
@@
 	(wire
 		(pts
-			(xy 190.5 97.79) (xy 167.64 97.79)
+			(xy 190.5 97.79) (xy 189.23 97.79)
 		)
 		(stroke
@@
 		)
 	)
+	(global_label "DP"
+		(shape input)
+		(at 191.77 105.41 0)
+		(fields_autoplaced yes)
+		(effects
+			(font
+				(size 1.27 1.27)
+			)
+			(justify left)
+		)
+		(property "Intersheetrefs" "${INTERSHEET_REFS}"
+			(at 197.2952 105.41 0)
+			(effects
+				(font
+					(size 1.27 1.27)
+				)
+				(justify left)
+				(hide yes)
+			)
+		)
+	)
 	(global_label "UART_TX"
 		(shape output)
@@
 			(effects
 				(font
+					(size 1.27 1.27)
+				)
+				(justify left)
+				(hide yes)
+			)
+		)
+	)
+	(global_label "DN"
+		(shape input)
+		(at 180.34 85.09 0)
+		(fields_autoplaced yes)
+		(effects
+			(font
+				(size 1.27 1.27)
+			)
+			(justify left)
+		)
+		(property "Intersheetrefs" "${INTERSHEET_REFS}"
+			(at 185.9257 85.09 0)
+			(effects
+				(font
