File: kicad/stm32f1/lnBMP_stm32_5pin_voltage_shifter2/output.kicad_sch (KiCad schematic)
At the start: 7 parts, among them J1 Debug port, J2 Debug port, J6 jtag, U2 3V->VTREF, U3 VTREF->3V, U4 VTREF<->3V

Commit message: beginning GD32 version
Parts:
- U2: footprint Voltshif -> Package_SO:VSSOP-8_2.3x2mm_P0.5mm
Changed lines of the file:
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@@
 			)
 		)
-		(property "Footprint" "Voltshif"
+		(property "Footprint" "Package_SO:VSSOP-8_2.3x2mm_P0.5mm"
 			(at 85.344 26.162 0)
 			(effects
@@
 					(size 1.27 1.27)
 				)
+				(hide yes)
 			)
 		)
