File: kicad/stm32f1/lnBMP_stm32_5pin_voltage_shifter2/powersupply.kicad_sch (KiCad schematic)
At the start: 17 parts, among them J3 USB, J9 Conn_01x03_Socket, U5 LM1117-3.3, U8 RT9013-33GB

Commit message: beginning GD32 version
Changed lines of the file:
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@@
 					(size 1.27 1.27)
 				)
+				(hide yes)
 			)
 		)
@@
 				)
 				(justify left)
+				(hide yes)
 			)
 		)
@@
 					(size 1.27 1.27)
 				)
+				(hide yes)
 			)
 		)
@@
 					(size 1.27 1.27)
 				)
+				(hide yes)
 			)
 		)
@@
 				)
 				(justify left)
-			)
-		)
+				(hide yes)
+			)
+		)

Commit message: first run at gd32 pcb with voltage shifter
Connections:
- net GND: now also C17.2, C18.2
Changed lines of the file:
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@@
+		)
+	)
+	(symbol
+		(lib_id "power:GND")
+		(at 30.48 154.94 0)
+		(unit 1)
+		(exclude_from_sim no)
+		(in_bom yes)
+		(on_board yes)
+		(dnp no)
+		(fields_autoplaced yes)
+		(property "Reference" "#PWR014"
+			(at 30.48 161.29 0)
+			(effects
+				(font
+					(size 1.27 1.27)
+				)
+				(hide yes)
+			)
+		)
+		(property "Value" "GND"
+			(at 30.48 160.02 0)
+			(effects
+				(font
+					(size 1.27 1.27)
+				)
+			)
+		)
+		(property "Footprint" ""
+			(at 30.48 154.94 0)
+			(effects
+				(font
+					(size 1.27 1.27)
+				)
+				(hide yes)
+			)
+		)
+		(property "Datasheet" ""
+			(at 30.48 154.94 0)
+			(effects
+				(font
+					(size 1.27 1.27)
+				)
+				(hide yes)
+			)
+		)
+		(property "Description" ""
+			(at 30.48 154.94 0)
+			(effects
+				(font
+					(size 1.27 1.27)
+				)
+				(hide yes)
+			)
+		)
+		(pin "1"
+		)
+		(instances
+			(project "lnBMP_stm32_voltage2"
+				(path "/fbe443d6-6d74-4abc-9dee-16e0160553bc/3e3374ff-17d6-414d-9a63-96aa322d3dc0"
+					(reference "#PWR014")
+					(unit 1)
+				)
+			)
 		)
 	)
