File: kicad/ch32v3x/lnBMP_ch32f_5pins_voltage_trans/lnBMP_ch32_revF_5pins_prot.kicad_pcb (KiCad board)
At the start: 2 copper layers, 49.8 x 33.3 mm, 65 parts, among them J1 jtag, J2 Conn_01x03_Socket, J2_DFU1 con2, J3 Debug port, J4 USB, J5 Debug port, U1 CH32V303RCT6, U2 LM1117-3.3, U3 3V->VTREF, U4 VTREF->3V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

Commit message: add 48° degrees rotated crystal
Parts:
- Y1: footprint Crystal:Crystal_SMD_TXC_7M-4Pin_3.2x2.5mm -> footprints:Crystal_SMD_TXC_7M-4Pin_3.2x2.5mm_45deg
- moved kibuzzard-671361D3 1.66 mm to (120.3, 82.3)
- moved C2 1.41 mm to (117.7, 83.7), turned to 180 degrees
- moved C3 0.71 mm to (117.7, 87.9), turned to 180 degrees
- moved Y1 0.45 mm to (120.9, 85.3)
Routing:
- net GND: track 278.4 -> 274.3 mm, vias 10 -> 12
- net Net-(U1-PF0): track 8.72 -> 6.24 mm, vias 2 -> 0
- net Net-(U1-PF1): track 9.06 -> 7.49 mm

Commit message: kicad: update to correct voltage translator footprint
Parts:
- removed the kibuzzard-65C1C789 at (114.7, 83.0)
- removed kibuzzard-65C1C7F5: G***, kibuzzard-65C1C7F5
- removed kibuzzard-65C1C805: G***, kibuzzard-65C1C805
- removed kibuzzard-6714B049: G***, kibuzzard-6714B049
- added kibuzzard-6731069B: G***, kibuzzard-6731069B, F.Cu at (115.0, 80.6)
- added kibuzzard-67310708: G***, kibuzzard-67310708, F.Cu at (114.9, 77.1)
- added kibuzzard-6731071F: G***, kibuzzard-6731071F, F.Cu at (114.9, 82.3)
- J3: value Debug port -> Dbg; footprint Connector_JST:JST_XH_B5B-XH-AM_1x05_P2.50mm_Vertical -> Connector_JST:JST_XH_B5B-XH-A_1x05_P2.50mm_Vertical
- U3, U4, U5: footprint Package_SO:VSSOP-8_2.3x2mm_P0.5mm -> Package_SO:TSSOP-8_3x3mm_P0.65mm
- moved RST1 4.81 mm to (131.6, 69.4)
- moved U6 4.51 mm to (122.8, 69.1)
- moved C10 3.99 mm to (117.8, 68.7), turned to 0 degrees
- moved R1 3.75 mm to (134.8, 76.1)
- moved J2_DFU1 3.11 mm to (135.3, 72.6), turned to 0 degrees
- moved C11 1.75 mm to (117.8, 70.3)
- moved U5 1.08 mm to (119.7, 73.0)
- moved kibuzzard-67137B47 0.80 mm to (114.9, 74.0)
- moved kibuzzard-671361D3 0.78 mm to (119.8, 82.9)
- moved U4 0.27 mm to (119.7, 80.6)
- moved kibuzzard-65C1C9D7 0.19 mm to (130.4, 72.4)
Routing:
- net +3.3V: track 179.6 -> 188.2 mm, vias 9 -> 11
- net V1.8: track 5.66 -> 11.3 mm, vias 0 -> 2
- net GND: track 274.3 -> 277.3 mm
- net VTREF: track 25.3 -> 22.7 mm
- net SWIO_DIR_3V: track 18.1 -> 20.6 mm
- net OUT_SWDCLK: track 22.3 -> 21.3 mm
- net INOUT_SWO: track 16.3 -> 15.4 mm
- net IN_FORCE_DFU: track 13.3 -> 13.8 mm
