File: kicad/gd32f303/swindle_gd32f303_revG/powersupply.kicad_sch (KiCad schematic)
At the start: 17 parts, among them J3 USB, J9 Conn_01x03_Socket, U5 LM1117-3.3, U8 RT9013-33GB

Commit message: update usb C connector + add 3 free pins
Parts:
- J3: footprint Connector_USB:USB_C_Receptacle_Palconn_UTC16-G -> Library:USB_C_Receptacle_Palconn_UTC16-G_no_hole
Changed lines of the file:
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@@
 			)
 		)
-		(property "Footprint" "Connector_USB:USB_C_Receptacle_Palconn_UTC16-G"
+		(property "Footprint" "Library:USB_C_Receptacle_Palconn_UTC16-G_no_hole"
 			(at 85.09 73.66 0)
 			(effects

Commit message: kicad: update GD32 PCB with SWDIO_DIR
Parts:
- J9: footprint Connector_PinHeader_1.27mm:PinHeader_1x03_P1.27mm_Vertical -> Connector_PinHeader_2.54mm:PinHeader_1x03_P2.54mm_Vertical
Changed lines of the file:
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@@
 			)
 		)
-		(property "Footprint" "Connector_PinHeader_1.27mm:PinHeader_1x03_P1.27mm_Vertical"
+		(property "Footprint" "Connector_PinHeader_2.54mm:PinHeader_1x03_P2.54mm_Vertical"
 			(at 166.37 144.78 0)
 			(effects
