File: kicad/gd32f303/swindle_gd32f303_revG/mcu.kicad_sch (KiCad schematic)
At the start: 16 parts, among them J4 DFU, J5 BOOT, U1 GD32F303, Y2 8Mhz

Commit message: update usb C connector + add 3 free pins
Parts:
- added J7: Conn_01x03_Pin, Connector_PinSocket_1.00mm:PinSocket_1x03_P1.00mm_Vertical, symbol Connector:Conn_01x04_Pin
Connections:
- net at U1.14 (PA4): now also J7.1 (Pin_1)
- net at U1.15 (PA5): now also J7.2 (Pin_2)
- net at U1.16 (PA6): now also J7.3 (Pin_3)
Changed lines of the file:
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@@
+	(wire
+		(pts
+			(xy 154.94 80.01) (xy 189.23 80.01)
+		)
+		(stroke
+			(width 0)
+			(type default)
+		)
+	)
 	(wire
 		(pts
@@
 	(wire
 		(pts
+			(xy 154.94 77.47) (xy 189.23 77.47)
+		)
+		(stroke
+			(width 0)
+			(type default)
+		)
+	)
+	(wire
+		(pts
 			(xy 198.12 96.52) (xy 198.12 97.79)
 		)
@@
 		(pts
 			(xy 104.14 88.9) (xy 119.38 88.9)
+		)
+		(stroke
+			(width 0)
+			(type default)
+		)
+	)
+	(wire
+		(pts
+			(xy 154.94 74.93) (xy 189.23 74.93)
 		)
 		(stroke
@@
 					(unit 1)
 				)
+			)
+		)
+	)
+	(symbol
+		(lib_id "Connector:Conn_01x04_Pin")
+		(at 194.31 77.47 0)
+		(mirror y)
+		(unit 1)
+		(exclude_from_sim no)
+		(in_bom yes)
+		(on_board yes)
+		(dnp no)
+		(property "Reference" "J7"
+			(at 193.675 69.85 0)
+			(effects
+				(font
+					(size 1.27 1.27)
+				)
+			)
+		)
+		(property "Value" "Conn_01x03_Pin"
+			(at 193.675 72.39 0)
+			(effects
+				(font
+					(size 1.27 1.27)
+				)
+				(hide yes)
+			)
+		)
+		(property "Footprint" "Connector_PinSocket_1.00mm:PinSocket_1x03_P1.00mm_Vertical"
+			(at 194.31 77.47 0)
+			(effects
+				(font
+					(size 1.27 1.27)
+				)
+				(hide yes)
+			)
+		)
+		(property "Datasheet" "~"
+			(at 194.31 77.47 0)
+			(effects
+				(font
+					(size 1.27 1.27)
+				)
+				(hide yes)
+			)
+		)
+		(property "Description" "Generic connector, single row, 01x04, script generated"
+			(at 194.31 77.47 0)
+			(effects
+				(font
+					(size 1.27 1.27)
+				)
+				(hide yes)
+			)
+		)
+		(pin "1"
+		)
+		(pin "4"
+		)
+		(pin "3"
+		)
+		(pin "2"
+		)
+		(instances
+			(project ""
+				(path "/fbe443d6-6d74-4abc-9dee-16e0160553bc/860eb7d0-1eba-4c3d-ac2c-5a3607b90fb5"
+					(reference "J7")
+					(unit 1)
+				)

Commit message: kicad: update GD32 PCB with SWDIO_DIR
Connections:
- net SWIO_DIR_3V: now reaches U1.2 (PC13)
Changed lines of the file:
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@@
 	(wire
 		(pts
-			(xy 119.38 88.9) (xy 119.38 77.47)
+			(xy 114.3 88.9) (xy 114.3 77.47)
 		)
 		(stroke
@@
 	(wire
 		(pts
-			(xy 119.38 77.47) (xy 121.92 77.47)
-		)
-		(stroke
-			(width 0)
-			(type default)
-		)
-	)
-	(wire
-		(pts
 			(xy 173.99 92.71) (xy 180.34 92.71)
 		)
@@
 	(wire
 		(pts
+			(xy 118.11 92.71) (xy 115.57 92.71)
+		)
+		(stroke
+			(width 0)
+			(type default)
+		)
+	)
+	(wire
+		(pts
 			(xy 189.23 105.41) (xy 191.77 105.41)
 		)
@@
 	(wire
 		(pts
+			(xy 121.92 82.55) (xy 118.11 82.55)
+		)
+		(stroke
+			(width 0)
+			(type default)
+		)
+	)
+	(wire
+		(pts
 			(xy 83.82 69.85) (xy 83.82 97.79)
 		)
@@
 	(wire
 		(pts
+			(xy 118.11 82.55) (xy 118.11 92.71)
+		)
+		(stroke
+			(width 0)
+			(type default)
+		)
+	)
+	(wire
+		(pts
 			(xy 116.84 113.03) (xy 121.92 113.03)
 		)
@@
 	(wire
 		(pts
+			(xy 114.3 77.47) (xy 121.92 77.47)
+		)
+		(stroke
+			(width 0)
+			(type default)
+		)
+	)
+	(wire
+		(pts
 			(xy 154.94 97.79) (xy 161.29 97.79)
 		)
@@
 	(wire
 		(pts
-			(xy 104.14 88.9) (xy 119.38 88.9)
+			(xy 104.14 88.9) (xy 114.3 88.9)
 		)
 		(stroke
@@
 				)
 				(justify left)
+				(hide yes)
+			)
+		)
+	)
+	(global_label "SWIO_DIR_3V"
+		(shape input)
+		(at 115.57 92.71 180)
+		(fields_autoplaced yes)
+		(effects
+			(font
+				(size 1.27 1.27)
+			)
+			(justify right)
+		)
+		(property "Intersheetrefs" "${INTERSHEET_REFS}"
+			(at 100.6105 92.71 0)
+			(effects
+				(font
+					(size 1.27 1.27)
+				)
+				(justify right)
 				(hide yes)
 			)
@@
 		)
 		(property "Value" "8Mhz"
-			(at 110.744 76.962 90)
-			(effects
-				(font
+			(at 106.172 73.406 90)
+			(effects
+				(font

Commit message: kicad: GD32, change the DIR pin to PA1
Connections:
- net SWIO_DIR_3V: now also U1.11 (PA1); no longer U1.2 (PC13)
Changed lines of the file:
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@@
 	(wire
 		(pts
-			(xy 118.11 92.71) (xy 115.57 92.71)
+			(xy 154.94 67.31) (xy 158.75 67.31)
 		)
 		(stroke
@@
 	(wire
 		(pts
+			(xy 158.75 63.5) (xy 166.37 63.5)
+		)
+		(stroke
+			(width 0)
+			(type default)
+		)
+	)
+	(wire
+		(pts
 			(xy 120.65 40.64) (xy 124.46 40.64)
 		)
@@
 		(pts
 			(xy 118.11 137.16) (xy 118.11 139.7)
+		)
+		(stroke
+			(width 0)
+			(type default)
+		)
+	)
+	(wire
+		(pts
+			(xy 158.75 67.31) (xy 158.75 63.5)
 		)
 		(stroke
@@
 		)
 	)
-	(global_label "SWIO_DIR_3V"
-		(shape input)
-		(at 115.57 92.71 180)
-		(fields_autoplaced yes)
-		(effects
-			(font
-				(size 1.27 1.27)
-			)
-			(justify right)
-		)
-		(property "Intersheetrefs" "${INTERSHEET_REFS}"
-			(at 100.6105 92.71 0)
-			(effects
-				(font
-					(size 1.27 1.27)
-				)
-				(justify right)
-				(hide yes)
-			)
-		)
-	)
 	(global_label "UART_TX"
 		(shape output)
@@
 			(effects
 				(font
+					(size 1.27 1.27)
+				)
+				(justify left)
+				(hide yes)
+			)
+		)
+	)
+	(global_label "SWIO_DIR_3V"
+		(shape input)
+		(at 166.37 63.5 0)
+		(fields_autoplaced yes)
+		(effects
+			(font
+				(size 1.27 1.27)
+			)
+			(justify left)
+		)
+		(property "Intersheetrefs" "${INTERSHEET_REFS}"
+			(at 181.3295 63.5 0)
+			(effects
+				(font

Commit message: update GD32 pcb
Parts:
- added J8: ~, Connector_PinSocket_1.27mm:PinSocket_1x05_P1.27mm_Vertical, symbol Connector:Conn_01x05_Pin
- J7: value Conn_01x03_Pin -> Conn_01x05_Pin; footprint Connector_PinSocket_1.00mm:PinSocket_1x03_P1.00mm_Vertical -> Connector_PinSocket_1.27mm:PinSocket_1x05_P1.27mm_Vertical; symbol Connector:Conn_01x04_Pin -> Connector:Conn_01x05_Pin
Connections:
- net GND: now also J7.5 (Pin_5)
- net PA4: now reaches U1.14 (PA4)
- net PA4: now also J8.1 (Pin_1); no longer J7.1 (Pin_1)
- net PA5: now reaches U1.15 (PA5)
- net PA5: now also J8.2 (Pin_2); no longer J7.2 (Pin_2)
- net PA6: now reaches U1.16 (PA6)
- net PA6: now also J8.3 (Pin_3); no longer J7.3 (Pin_3)
- net PB7: now reaches J7.4 (Pin_4)
- net PB7: now also U1.43 (PB7)
- net PA7: now reaches U1.17 (PA7)
- net PA7: now also J8.4 (Pin_4)
- net PB0: now reaches U1.18 (PB0)
- net PB0: now also J8.5 (Pin_5)
- net PB3: now reaches U1.39 (PB3)
- net PB3: now also J7.1 (Pin_1)
- net PB4: now reaches U1.40 (PB4)
- net PB4: now also J7.2 (Pin_2)
- net PB5: now reaches U1.41 (PB5)
- net PB5: now also J7.3 (Pin_3)
