File: kicad/ch32v3x/swindle_revI/swindle_ch32_revI.kicad_pcb (KiCad board)
At the start: 2 copper layers, 49.8 x 33.3 mm, 64 parts, among them J1 jtag, J2 Conn_01x03_Socket, J2_DFU1 con2, J3 Dbg, J4 USB, J5 Debug port, U1 CH32V303RCT6, U2 LM1117-3.3, U3 3V->VTREF, U4 VTREF->3V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

Commit message: kicad : update ch32 to revI
Parts:
- removed kibuzzard-65D8420C: G***, kibuzzard-65D8420C
- removed kibuzzard-679335ED: G***, kibuzzard-679335ED
- added kibuzzard-67ECD764: G***, kibuzzard-67ECD764, F.Cu at (149.7, 99.1)
- added kibuzzard-67ECD9AB: G***, kibuzzard-67ECD9AB, F.Cu at (131.1, 77.7)
- J3: footprint Connector_JST:JST_XH_B5B-XH-A_1x05_P2.50mm_Vertical -> Connector_PinSocket_1.27mm:PinSocket_1x05_P1.27mm_Vertical
- moved J2 14.1 mm to (126.1, 68.6)
- moved C11 13.0 mm to (130.7, 68.6), turned to 90 degrees
- moved U6 11.3 mm to (134.0, 68.9)
- moved RST1 9.01 mm to (139.7, 73.4), turned to -90 degrees
- moved kibuzzard-65C1C789 8.05 mm to (140.4, 79.0)
- moved kibuzzard-65C1C8EE 7.41 mm to (140.4, 80.3)
- moved kibuzzard-65C1C918 6.37 mm to (140.4, 81.6)
- moved kibuzzard-65C1C92F 6.10 mm to (140.4, 82.9)
- moved C10 4.98 mm to (122.7, 67.8)
- moved kibuzzard-65C1C972 3.78 mm to (140.5, 84.2)
- moved kibuzzard-65C1C9D7 2.38 mm to (132.3, 73.9)
- moved U5 1.85 mm to (119.8, 71.1)
- moved J3 1.81 mm to (143.5, 82.4), turned to 180 degrees
- moved U3 0.98 mm to (119.7, 75.8)
Routing:
- net +3.3V: track 188.2 -> 174.1 mm, vias 11 -> 8
- net GND: track 277.3 -> 265.0 mm, vias 12 -> 14
- net V1.8: track 11.3 -> 4.59 mm, vias 2 -> 0
- net NRESET: track 56.9 -> 51.0 mm, vias 2 -> 3
- net VTREF: track 22.7 -> 17.0 mm, vias 4 -> 3
- net SWIO_DIR_3V: track 24.6 -> 22.0 mm
- net SWDIO: track 11.3 -> 8.84 mm
- net OUT_SWDIO_3V: track 11.3 -> 13.4 mm
- net UART_TX: track 11.3 -> 10.2 mm
- net OUT_SWDIO: track 24.9 -> 26.0 mm
- net OUT_SWDCLK: track 21.3 -> 21.9 mm
