File: kicad/ch32v3x/swindle_revI/swindle_ch32_revI.kicad_sch (KiCad schematic)
At the start: 34 parts, among them J1 jtag, J2 Conn_01x03_Socket, J2_DFU1 con2, J3 Dbg, J4 USB, J5 Debug port, U1 CH32V303RCT6, U2 LM1117-3.3, U3 3V->VTREF, U4 VTREF->3V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

Commit message: kicad : update ch32 to revI
Parts:
- J3: footprint Connector_JST:JST_XH_B5B-XH-A_1x05_P2.50mm_Vertical -> Connector_PinSocket_1.27mm:PinSocket_1x05_P1.27mm_Vertical
Changed lines of the file:
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@@
 				)
 				(justify left)
+				(hide yes)
 			)
 		)
@@
 			)
 		)
-		(property "Footprint" "Connector_JST:JST_XH_B5B-XH-A_1x05_P2.50mm_Vertical"
+		(property "Footprint" "Connector_PinSocket_1.27mm:PinSocket_1x05_P1.27mm_Vertical"
 			(at 143.51 161.29 90)
 			(effects
@@
 					(size 1.27 1.27)
 				)
-			)
-		)
+				(hide yes)
+			)
+		)
