File: kicad/rp2040_zero/rev1_no_voltage/zero_r1_no_vt.kicad_pcb (KiCad board)
At the start: 2 copper layers, 39.7 x 30.2 mm, 18 parts, among them J1 jtag, J3 Debug port, J5 Debug port, U1 RP2040-Zero

Commit message: rp2040: update pcb, add optional pullup
Parts:
- added PULLUP: R_0603_1608Metric, Resistor_SMD:R_0603_1608Metric, F.Cu at (122.5, 78.3)
- added PULLUP2: R_0603_1608Metric, Resistor_SMD:R_0603_1608Metric, F.Cu at (122.5, 81.1)
Routing:
- net +3.3V: track 0.00 -> 31.7 mm, vias 0 -> 2
- net OUT_UART_RX_3V: track 22.7 -> 23.6 mm
- net GND: vias 7 -> 11
