File: kicad/ch32v3x/swindle_revJ/swindle_ch32_revJ.kicad_sch (KiCad schematic)
At the start: 34 parts, among them J1 jtag, J2 Conn_01x03_Socket, J2_DFU1 con2, J3 Dbg, J4 USB, J5 Debug port, U1 CH32V303RCT6, U2 LM1117-3.3, U3 3V->VTREF, U4 VTREF->3V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

Commit message: update CH32 pcb
Parts:
- removed C10, C11, C5: 100n, Resistor_SMD:R_0603_1608Metric, symbol Device:C_Small
- removed C4: 100u, Capacitor_SMD:C_1206_3216Metric_Pad1.33x1.80mm_HandSolder, symbol Device:C_Polarized
- removed D2: LED, Diode_SMD:D_0805_2012Metric, symbol Device:LED
- removed J1: jtag, Connector_PinHeader_1.27mm:PinHeader_2x05_P1.27mm_Vertical_SMD, symbol Connector:Conn_ARM_JTAG_SWD_10
- removed J2: Conn_01x03_Socket, Connector_PinHeader_2.54mm:PinHeader_1x03_P2.54mm_Vertical, symbol Connector:Conn_01x03_Socket
- removed J3: Dbg, Connector_PinSocket_1.27mm:PinSocket_1x05_P1.27mm_Vertical, symbol Connector:Conn_01x05_Male
- removed J4: USB, Connector_USB:USB_C_Receptacle_Palconn_UTC16-G, symbol Connector:USB_C_Receptacle
- removed J5: Debug port, Connector_JST:JST_XH_B5B-XH-A_1x05_P2.50mm_Vertical, symbol Connector:Conn_01x05_Male
- removed R4, R6: 5.1k, Resistor_SMD:R_0603_1608Metric, symbol Device:R_Small
- removed R7: 330, Resistor_SMD:R_0603_1608Metric, symbol Device:R_Small
- removed U2: LM1117-3.3, Package_TO_SOT_SMD:SOT-223, symbol Regulator_Linear:LM1117-3.3
- removed U3: 3V->VTREF, Package_SO:TSSOP-8_3x3mm_P0.65mm, symbol Logic_LevelTranslator:SN74LVC2T45DCUR
- removed U4: VTREF->3V, Package_SO:TSSOP-8_3x3mm_P0.65mm, symbol Logic_LevelTranslator:SN74LVC2T45DCUR
- removed U5: VTREF<->3V, Package_SO:TSSOP-8_3x3mm_P0.65mm, symbol Logic_LevelTranslator:SN74LVC2T45DCUR
- removed U6: RT9013-33GB, PCM_Package_TO_SOT_SMD_AKL:TSOT-23-5, symbol 2024-10-20_09-04-45:RT9013-33GB
Connections:
- net PA0: now reaches U1.14 (PA0)
- net PA1: now reaches U1.15 (PA1)
- net PA2: now reaches U1.16 (PA2)
- net PA5: now reaches U1.21 (PA5)
- net PA6: now reaches U1.22 (PA6)
- net PA7: now reaches U1.23 (PA7)
- net PB0: now reaches U1.26 (PB0)
- net PB1: now reaches U1.27 (PB1)
- net PB15: now reaches U1.36 (PB15)
- net PC6: now reaches U1.37 (PC6)
- net PC7: now reaches U1.38 (PC7)
- net PC8: now reaches U1.39 (PC8)
- net PC9: now reaches U1.40 (PC9)
- net PB3: now reaches U1.55 (PB3)
- net PB4: now reaches U1.56 (PB4)
- net PB5: now reaches U1.57 (PB5)
Other:
- added sheet Connectors (untitled.kicad_sch)
- added sheet usb (usb.kicad_sch)
- added sheet voltage_translators (vt.kicad_sch)
- moved on the sheet: C6, C7, C8, C9

Commit message: kicad: update new wch
Changed lines of the file:
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@@
 					(size 1.27 1.27)
 				)
+				(hide yes)
 			)
 		)
