File: kicad/ch32v3x/swindle_revJ/swindle_ch32_revJ.kicad_sch (KiCad schematic)
At the start: 16 parts, among them J2_DFU1 con2, U1 CH32V303RCT6, Y1 8Mhz

Commit message: Kicad update: ch32: update pcb , add boot pin control ch32: Ground PB2 so that the internal bootloader is on USB rp_zero_mini :add mostfet to rp zero mini
general update
Connections:
- net GND: now also U1.28 (PB2)
