File: kicad/gd32f303/swindle_gd32f303_revG_mini/output.kicad_sch (KiCad schematic)
At the start: 2 parts, among them J1 Debug port, J2 Debug port

Commit message: kicad: order to pcbway
Connections:
- net INOUT_NRESET_3V renamed INOUT_NRESET
Changed lines of the file:
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@@
+	(wire
+		(pts
+			(xy 43.18 157.48) (xy 71.12 157.48)
+		)
+		(stroke
+			(width 0)
+			(type default)
+		)
+	)
 	(wire
 		(pts
@@
 		)
 	)
+	(global_label "INOUT_NRESET"
+		(shape bidirectional)
+		(at 71.12 157.48 0)
+		(fields_autoplaced yes)
+		(effects
+			(font
+				(size 1.27 1.27)
+			)
+			(justify left)
+		)
+		(property "Intersheetrefs" "${INTERSHEET_REFS}"
+			(at 87.1402 157.4006 0)
+			(effects
+				(font
+					(size 1.27 1.27)
+				)
+				(justify left)
+				(hide yes)
+			)
+		)
+	)
 	(global_label "OUT_UART_RX_3V"
 		(shape input)
@@
 			(effects
 				(font
+					(size 1.27 1.27)
+				)
+				(justify right)
+				(hide yes)
+			)
+		)
+	)
+	(global_label "INOUT_NRESET_3V"
+		(shape bidirectional)
+		(at 43.18 157.48 180)
+		(fields_autoplaced yes)
+		(effects
+			(font
+				(size 1.27 1.27)
+			)
+			(justify right)
+		)
+		(property "Intersheetrefs" "${INTERSHEET_REFS}"
+			(at 22.2107 157.48 0)
+			(effects
+				(font
