File: kicad/rp2040_zero/rev2_mini/zero_r2_mini.kicad_pcb (KiCad board)
At the start: 2 copper layers, 34.6 x 28.3 mm, 12 parts, among them J3 Debug port, J5 Debug port, U1 RP2040-Zero

Commit message: kicad: RP mini , add reset mosfet
Parts:
- added Q1: DMG2302U, Package_TO_SOT_SMD:SOT-23, F.Cu at (119.8, 70.8)
- added R1: 1k, Resistor_SMD:R_0603_1608Metric, F.Cu at (116.7, 70.5)
- added R2: 330, Resistor_SMD:R_0603_1608Metric, F.Cu at (123.0, 70.5)
Connections:
- U1 pad 22: INOUT_NRESET -> DRIVE_RESET
Routing:
- net DRIVE_RESET: track 0.00 -> 23.2 mm, vias 0 -> 1
- net INOUT_NRESET: track 31.9 -> 22.2 mm, vias 1 -> 0
- net Net-(Q1-D): track 0.00 -> 2.62 mm
