File: kicad/rp2040_zero/rev2/zero_r2.kicad_pcb (KiCad board)
At the start: 2 copper layers, 41.8 x 30.2 mm, 31 parts, among them J1 jtag, J2 Conn_01x03_Socket, J3 Debug port, J5 Debug port, U1 RP2040-Zero, U3 3V->VTREF, U4 VTREF->3V, U5 VTREF<->3V, U6 RT9013-33GB

Commit message: Kicad update: ch32: update pcb , add boot pin control ch32: Ground PB2 so that the internal bootloader is on USB rp_zero_mini :add mostfet to rp zero mini
general update
Parts:
- removed PULLUP, PULLUP2: R_0603_1608Metric, Resistor_SMD:R_0603_1608Metric
- removed kibuzzard-67310D89: G***, kibuzzard-67310D89
- removed kibuzzard-67310DA4: G***, kibuzzard-67310DA4
- removed kibuzzard-67A3B7A3: G***, kibuzzard-67A3B7A3
- removed kibuzzard-67D71DD3: G***, kibuzzard-67D71DD3
- removed kibuzzard-67D71DDE: G***, kibuzzard-67D71DDE
- removed kibuzzard-6845954C: G***, kibuzzard-6845954C
- added Q1: DMG2302U, Package_TO_SOT_SMD:SOT-23, F.Cu at (117.9, 68.4)
- added R1: 10k, Resistor_SMD:R_0603_1608Metric, F.Cu at (117.9, 81.8)
- added R2: 1k, Resistor_SMD:R_0603_1608Metric, F.Cu at (117.9, 71.4)
- added R3: 330, Resistor_SMD:R_0603_1608Metric, F.Cu at (114.2, 67.3)
- added kibuzzard-6A64D073: G***, kibuzzard-6A64D073, F.Cu at (113.2, 86.0)
- added kibuzzard-6A64D231: G***, kibuzzard-6A64D231, F.Cu at (110.7, 95.2)
- U6: footprint PCM_Package_TO_SOT_SMD_AKL:TSOT-23-5 -> Package_TO_SOT_SMD:SOT-23-5_HandSoldering
- kibuzzard-67D71D53: moved to B.Cu
- moved kibuzzard-6719D703 7.16 mm to (112.7, 93.1)
- moved kibuzzard-6714FCCA 0.40 mm to (127.5, 72.2)
- moved C1 0.38 mm to (121.3, 68.0)
- moved J1 0.35 mm to (119.5, 91.8)
- moved U4 0.34 mm to (121.0, 84.8)
- moved C3 0.31 mm to (121.2, 69.7)
- moved C11 0.11 mm to (117.2, 84.1)
Connections:
- U1 pad 22: INOUT_NRESET -> INOUT_NRESET_3V
Routing:
- net GND: track 110.5 -> 57.9 mm, vias 17 -> 25
- net INOUT_NRESET_3V: track 0.00 -> 25.5 mm, vias 0 -> 4
- net INOUT_NRESET: track 71.5 -> 63.3 mm, vias 5 -> 3
- net VTREF: track 47.3 -> 40.8 mm, vias 0 -> 1
- net INOUT_SWO: track 0.00 -> 6.28 mm
- net Net-(Q1-D): track 0.00 -> 2.92 mm
- net OUT_UART_RX: track 11.9 -> 14.4 mm
- net SWIO_DIR_3V: track 12.4 -> 14.1 mm
- net OUT_SWDCLK_3V: track 9.44 -> 10.9 mm, vias 2 -> 1
