File: kicad/rp2040_zero/rev2_w5500/w5500b.kicad_sch (KiCad schematic)
At the start: 40 parts, among them P4 J1B1211CCD, U5 W5500, Y4 25MHz

Commit message: w5500 : update 1
Connections:
- net 3V3: no longer R14.2
- net ACTn: now also R47.1; no longer R47.2
- net LINKn: now also R32.1; no longer R32.2
- net at P4.11 (YLED_K): now also R47.2; no longer R47.1
- net at P4.9 (GLED_K): now also R32.2; no longer R32.1
- net SPI0_CSn renamed CSn
- net SPI0_RX renamed MISO
- net SPI0_SCK renamed CLK
- net SPI0_TX renamed MOSI
Other:
- moved on the sheet: C66, C67, R14, R32, R47, R57, R58, R59, Y4

Commit message: preliminary W5500
Parts:
- L1: footprint IND-0603 -> Inductor_SMD:L_0603_1608Metric
- Y4: footprint OSC-82J0626 -> Crystal:Crystal_SMD_TXC_7M-4Pin_3.2x2.5mm
Connections:
- net 3V3: now also R14.2
- net CHGND renamed SH
- net INTn renamed W5INTn
- net RSTn renamed W5RSTn
Other:
- moved on the sheet: R50
Changed lines of the file:
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@@
 	)
 	(junction
-		(at 113.03 101.6)
+		(at 114.3 101.6)
 		(diameter 0)
 		(color 0 0 0 0)
@@
 	(wire
 		(pts
-			(xy 110.49 116.84) (xy 113.03 116.84)
+			(xy 110.49 116.84) (xy 114.3 116.84)
 		)
 		(stroke
@@
 	(wire
 		(pts
+			(xy 190.5 73.66) (xy 194.31 73.66)
+		)
+		(stroke
+			(width 0)
+			(type default)
+		)
+	)
+	(wire
+		(pts
 			(xy 140.97 35.56) (xy 148.59 35.56)
 		)
@@
 	(wire
 		(pts
-			(xy 194.31 73.66) (xy 191.77 73.66)
-		)
-		(stroke
-			(width 0)
-			(type default)
-		)
-	)
-	(wire
-		(pts
 			(xy 85.09 99.06) (xy 87.63 99.06)
 		)
@@
 	(wire
 		(pts
-			(xy 113.03 116.84) (xy 113.03 111.76)
+			(xy 114.3 116.84) (xy 114.3 111.76)
 		)
 		(stroke
@@
 	(wire
 		(pts
-			(xy 118.11 101.6) (xy 113.03 101.6)
+			(xy 118.11 101.6) (xy 114.3 101.6)
 		)
 		(stroke
@@
 	(wire
 		(pts
-			(xy 113.03 101.6) (xy 113.03 104.14)
+			(xy 114.3 101.6) (xy 114.3 104.14)
 		)
 		(stroke
@@
 	(wire
 		(pts
-			(xy 113.03 101.6) (xy 105.41 101.6)
+			(xy 105.41 101.6) (xy 114.3 101.6)
 		)
 		(stroke
@@
 		)
 	)
-	(global_label "RSTn"
+	(global_label "W5RSTn"
 		(shape input)
 		(at 181.61 66.04 0)
@@
 		)
 		(property "Intersheetrefs" "${INTERSHEET_REFS}"
-			(at 189.1913 66.04 0)
+			(at 191.8522 66.04 0)
 			(hide yes)
 			(show_name no)
@@
 		)
 	)
-	(global_label "INTn"
+	(global_label "W5INTn"
 		(shape output)
 		(at 214.63 88.9 0)
@@
 		)
 		(property "Intersheetrefs" "${INTERSHEET_REFS}"
-			(at 221.6671 88.9 0)
+			(at 224.328 88.9 0)
 			(hide yes)
 			(show_name no)
@@
 			)
 		)
-		(property "Footprint" "IND-0603"
+		(property "Footprint" "Inductor_SMD:L_0603_1608Metric"
 			(at 153.67 25.4 0)
 			(hide yes)
@@
 		(dnp no)
 		(property "Reference" "R49"
-			(at 110.49 104.14 90)
+			(at 111.252 104.14 90)
 			(show_name no)
 			(do_not_autoplace no)
@@
 		)
 		(property "Value" "49.9R"
-			(at 110.49 109.22 90)
+			(at 111.252 109.22 90)
 			(show_name no)
 			(do_not_autoplace no)
@@
 			)
 		)
-		(property "Value" "CHGND"
+		(property "Value" "SH"
 			(at 54.61 135.89 0)
 			(show_name no)
@@
 	(symbol
 		(lib_id "Scott_lib:RES-0402")
-		(at 113.03 109.22 180)
+		(at 114.3 109.22 180)
 		(unit 1)
 		(body_style 1)
@@
 		(dnp no)
 		(property "Reference" "R50"
-			(at 113.03 104.14 90)
+			(at 115.57 104.394 90)
 			(show_name no)
 			(do_not_autoplace no)
@@
 		)
 		(property "Value" "49.9R"
-			(at 113.03 109.22 90)
+			(at 115.57 109.22 90)
 			(show_name no)
 			(do_not_autoplace no)
@@
 		)
 		(property "Footprint" "Resistor_SMD:R_0603_1608Metric"
-			(at 113.03 109.22 0)
+			(at 114.3 109.22 0)
 			(hide yes)
 			(show_name no)
@@
 		)
 		(property "Datasheet" ""
-			(at 113.03 109.22 0)
+			(at 114.3 109.22 0)
 			(hide yes)
 			(show_name no)
@@
 		)
 		(property "Description" "RES-0402"
-			(at 113.03 109.22 0)
+			(at 114.3 109.22 0)
 			(hide yes)
 			(show_name no)
@@
 		(property "Value" "25MHz"
 			(at 247.65 116.84 90)
+			(hide yes)
 			(show_name no)
 			(do_not_autoplace no)
@@
 			)
 		)
-		(property "Footprint" "OSC-82J0626"
+		(property "Footprint" "Crystal:Crystal_SMD_TXC_7M-4Pin_3.2x2.5mm"
 			(at 248.92 111.76 0)
 			(hide yes)
