File: kicad/ch32v3x/swindle_revJ_mini/swindle_ch32_revJ_mini.kicad_pcb (KiCad board)
At the start: 2 copper layers, 38.3 x 34 mm, 56 parts, among them J10 Debug port, J2_DFU1 con2, J3 Dbg, J4 USB, J5 Debug port, J6 Debug port, J7 Conn_01x03_Pin, J8 Debug port, J9 Conn_01x03_Pin, Q1-A2SHB1 DMG2302U, U1 CH32V303RCT6, U2 LM1117-3.3, Y1 8Mhz

Commit message: Kicad update: ch32: update pcb , add boot pin control ch32: Ground PB2 so that the internal bootloader is on USB rp_zero_mini :add mostfet to rp zero mini
general update
Parts:
- removed J9: Conn_01x03_Pin, Connector_PinSocket_1.27mm:PinSocket_1x03_P1.27mm_Vertical
- removed the kibuzzard-65C1C918 at (125.2, 73.5)
- removed the kibuzzard-65C1C92F at (125.3, 72.3)
- removed the kibuzzard-65C1C972 at (125.3, 70.1)
- removed kibuzzard-67ECD9AB: G***, kibuzzard-67ECD9AB
- removed kibuzzard-68977CD7: G***, kibuzzard-68977CD7
- added J3_BL1: con2, Connector_PinHeader_1.27mm:PinHeader_1x02_P1.27mm_Vertical, F.Cu at (127.9, 74.4)
- added kibuzzard-6A634FB9: G***, kibuzzard-6A634FB9, F.Cu at (124.9, 69.1)
- added kibuzzard-6A635004: G***, kibuzzard-6A635004, F.Cu at (125.1, 73.5)
- added kibuzzard-6A635025: G***, kibuzzard-6A635025, F.Cu at (125.0, 72.3)
- added kibuzzard-6A635259: G***, kibuzzard-6A635259, F.Cu at (128.5, 76.2)
- added kibuzzard-6A635294: G***, kibuzzard-6A635294, F.Cu at (147.6, 66.0)
- moved R9 2.57 mm to (132.2, 74.1), turned to 0 degrees
- moved R11 0.64 mm to (127.6, 70.8), turned to 180 degrees
Connections:
- U1 pad 28: unconnected-(U1-PB2-Pad28) -> GND
Routing:
- net PB3: track 7.30 -> 0.00 mm
- net PB5: track 6.21 -> 0.00 mm
- net +3.3V: track 129.0 -> 132.3 mm
- net Net-(J3_BL1-Pin_2): track 8.75 -> 10.9 mm
- net INOUT_NRESET: track 42.9 -> 41.0 mm
- net PB4: track 12.7 -> 11.0 mm, vias 1 -> 0
- net GND: track 133.2 -> 132.6 mm, vias 22 -> 26
- net IN_FORCE_DFU: track 14.3 -> 15.0 mm, vias 0 -> 1
- net DRIVE_RESET: track 15.8 -> 16.4 mm, vias 2 -> 0

Commit message: kicad: update ch32 with the pullup
Parts:
- removed kibuzzard-6A635294: G***, kibuzzard-6A635294
- added R12: 1k, Resistor_SMD:R_0603_1608Metric, F.Cu at (124.9, 73.3)
- added kibuzzard-6AB8B403: G***, kibuzzard-6AB8B403, F.Cu at (147.6, 66.0)
- moved kibuzzard-6A635004 1.57 mm to (125.1, 75.1)
- moved kibuzzard-65C1C8EE 0.72 mm to (125.3, 76.5)
- moved kibuzzard-6A635025 0.71 mm to (125.0, 71.6)
- moved J3_BL1 0.41 mm to (128.3, 74.4)
Routing:
- net OUT_UART_RX: track 29.1 -> 35.5 mm
- net +3.3V: track 132.3 -> 137.1 mm
- net GND: track 132.6 -> 130.5 mm, vias 26 -> 30
- net INOUT_NRESET: track 41.0 -> 39.4 mm
- net OUT_SWDIO: track 12.6 -> 11.6 mm
